File: Hardware/SparkFun_PIR_Breakout.sch (EAGLE design)
At the start: 11 parts, among them U1 EKMC4607112k

Commit message: post checklist changes
Parts:
- added C1: 0.1uF, SparkFun-Capacitors:0.1UF-0603-25V-(+80/-20%)
- added D1: 24V, SparkFun-DiscreteSemi:DIODE_TVS
- added H1: STAND-OFF, SparkFun-Hardware:STAND-OFF
- LOGO3: value SFE_LOGO_NAME.1_INCH -> SFE_LOGO_NAME_FLAME.1_INCH; device SparkFun-Aesthetics:SFE_LOGO_NAME.1_INCH -> SparkFun-Aesthetics:SFE_LOGO_NAME_FLAME.1_INCH
Connections:
- net 3.3V: now also C1.1, D1.C
- net GND: now also C1.2, D1.A
Changed lines of the file:
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@@
 <part name="JP8" library="SparkFun" deviceset="FIDUCIAL" device="UFIDUCIAL"/>
 <part name="JP9" library="SparkFun" deviceset="FIDUCIAL" device="UFIDUCIAL"/>
-<part name="LOGO3" library="SparkFun-Aesthetics" deviceset="SFE_LOGO_NAME" device=".1_INCH"/>
+<part name="LOGO3" library="SparkFun-Aesthetics" deviceset="SFE_LOGO_NAME_FLAME" device=".1_INCH"/>
 <part name="LOGO4" library="SparkFun-Aesthetics" deviceset="SFE_LOGO_FLAME" device=".1_INCH"/>
 <part name="U1" library="SparkFun-Sensors" deviceset="PIR_EKM" device="4607112K" value="EKMC4607112k"/>
@@
 <part name="GND1" library="SparkFun" deviceset="GND" device=""/>
 <part name="SUPPLY2" library="SparkFun-PowerSymbols" deviceset="3.3V" device=""/>
+<part name="D1" library="SparkFun-DiscreteSemi" deviceset="DIODE_TVS" device="" value="24V"/>
+<part name="C1" library="SparkFun-Capacitors" deviceset="0.1UF" device="-0603-25V-(+80/-20%)" value="0.1uF"/>
+<part name="SUPPLY3" library="SparkFun-PowerSymbols" deviceset="3.3V" device=""/>
+<part name="GND3" library="SparkFun" deviceset="GND" device=""/>
+<part name="H1" library="SparkFun-Hardware" deviceset="STAND-OFF" device=""/>
 </parts>
 <sheets>
@@
 <attribute name="VALUE" x="170.18" y="99.314" size="1.778" layer="96" font="vector" align="bottom-center"/>
 </instance>
+<instance part="D1" gate="G$1" x="71.12" y="91.44" smashed="yes" rot="R90">
+<attribute name="NAME" x="69.088" y="87.63" size="1.778" layer="95" font="vector" rot="R90"/>
+<attribute name="VALUE" x="73.152" y="87.63" size="1.778" layer="96" font="vector" rot="R90" align="top-left"/>
+</instance>
+<instance part="C1" gate="G$1" x="78.74" y="88.9" smashed="yes">
+<attribute name="NAME" x="80.264" y="91.821" size="1.778" layer="95" font="vector"/>
+<attribute name="VALUE" x="80.264" y="86.741" size="1.778" layer="96" font="vector"/>
+</instance>
+<instance part="SUPPLY3" gate="G$1" x="76.2" y="101.6" smashed="yes">
+<attribute name="VALUE" x="76.2" y="104.394" size="1.778" layer="96" font="vector" align="bottom-center"/>
+</instance>
+<instance part="GND3" gate="1" x="76.2" y="78.74" smashed="yes" rot="MR0">
+<attribute name="VALUE" x="78.74" y="76.2" size="1.778" layer="96" font="vector" rot="MR0"/>
+</instance>
+<instance part="H1" gate="G$1" x="243.84" y="30.48" smashed="yes"/>
 </instances>
 <busses>
@@
 <wire x1="170.18" y1="88.9" x2="170.18" y2="86.36" width="0.1524" layer="91"/>
 </segment>
+<segment>
+<pinref part="D1" gate="G$1" pin="A"/>
+<wire x1="71.12" y1="86.36" x2="71.12" y2="83.82" width="0.1524" layer="91"/>
+<wire x1="71.12" y1="83.82" x2="76.2" y2="83.82" width="0.1524" layer="91"/>
+<pinref part="C1" gate="G$1" pin="2"/>
+<wire x1="76.2" y1="83.82" x2="78.74" y2="83.82" width="0.1524" layer="91"/>
+<wire x1="78.74" y1="83.82" x2="78.74" y2="86.36" width="0.1524" layer="91"/>
+<wire x1="76.2" y1="83.82" x2="76.2" y2="81.28" width="0.1524" layer="91"/>
+<junction x="76.2" y="83.82"/>
+<pinref part="GND3" gate="1" pin="GND"/>
+</segment>
 </net>
 <net name="3.3V" class="0">
@@
 <wire x1="170.18" y1="93.98" x2="170.18" y2="96.52" width="0.1524" layer="91"/>
 </segment>
+<segment>
+<pinref part="C1" gate="G$1" pin="1"/>
+<wire x1="78.74" y1="93.98" x2="78.74" y2="99.06" width="0.1524" layer="91"/>
+<wire x1="78.74" y1="99.06" x2="76.2" y2="99.06" width="0.1524" layer="91"/>
+<pinref part="D1" gate="G$1" pin="C"/>
+<wire x1="76.2" y1="99.06" x2="71.12" y2="99.06" width="0.1524" layer="91"/>
+<wire x1="71.12" y1="99.06" x2="71.12" y2="96.52" width="0.1524" layer="91"/>
+<wire x1="76.2" y1="99.06" x2="76.2" y2="101.6" width="0.1524" layer="91"/>
+<junction x="76.2" y="99.06"/>
+<pinref part="SUPPLY3" gate="G$1" pin="3.3V"/>
+</segment>
 </net>

Commit message: checklist saved changes
Other:
- note added: "This PIR sensor is different between 170 uA (IC-15368) and 1uA (IC-15370) versions"
Changed lines of the file:
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@@
 <text x="109.22" y="132.08" size="2.54" layer="94" font="vector">PIR Breakout</text>
 <text x="109.22" y="129.54" size="1.27" layer="94" font="vector">VIN: 2.3V-4.0V</text>
+<text x="101.6" y="71.12" size="1.27" layer="97" font="vector">This PIR sensor is different
+between 170 uA (IC-15368)
+and 1uA (IC-15370) versions</text>
 </plain>
 <instances>
@@
 </schematic>
 </drawing>
+<compatibility>
+<note version="6.3" minversion="6.2.2" severity="warning">
+Since Version 6.2.2 text objects can contain more than one line,
+which will not be processed correctly with this version.
+</note>
+</compatibility>
 </eagle>
