File: Production/SEN-17373/SparkFun_PIR_Breakout-Panel.brd (EAGLE design)
At the start: 204.5 x 124.2 mm, 1546 parts, among them U1 EKMC4607112k, U10 EKMC4607112k, U11 EKMC4607112k, U12 EKMC4607112k, U13 EKMC4607112k, U14 EKMC4607112k, U15 EKMC4607112k, U16 EKMC4607112k, U17 EKMC4607112k, U18 EKMC4607112k, U19 EKMC4607112k, U2 EKMC4607112k, U20 EKMC4607112k, U21 EKMC4607112k, U22 EKMC4607112k, U23 EKMC4607112k, U24 EKMC4607112k, U25 EKMC4607112k, U26 EKMC4607112k, U27 EKMC4607112k, U28 EKMC4607112k, U29 EKMC4607112k, U3 EKMC4607112k, U30 EKMC4607112k, U31 EKMC4607112k, U32 EKMC4607112k, U33 EKMC4607112k, U34 EKMC4607112k, U35 EKMC4607112k, U36 EKMC4607112k, U37 EKMC4607112k, U38 EKMC4607112k, U39 EKMC4607112k, U4 EKMC4607112k, U40 EKMC4607112k, U41 EKMC4607112k, U42 EKMC4607112k, U43 EKMC4607112k, U44 EKMC4607112k, U45 EKMC4607112k, U46 EKMC4607112k, U47 EKMC4607112k, U48 EKMC4607112k, U49 EKMC4607112k, U5 EKMC4607112k, U50 EKMC4607112k, U51 EKMC4607112k, U52 EKMC4607112k, U53 EKMC4607112k, U54 EKMC4607112k, U55 EKMC4607112k, U56 EKMC4607112k, U57 EKMC4607112k, U58 EKMC4607112k, U59 EKMC4607112k, U6 EKMC4607112k, U60 EKMC4607112k, U61 EKMC4607112k, U62 EKMC4607112k, U63 EKMC4607112k, U64 EKMC4607112k, U65 EKMC4607112k, U66 EKMC4607112k, U67 EKMC4607112k, U68 EKMC4607112k, U69 EKMC4607112k, U7 EKMC4607112k, U70 EKMC4607112k, U8 EKMC4607112k, U9 EKMC4607112k

Commit message: updating panel file
Parts:
- removed C61, C62, C63, C64, C65, C66, C67, C68, C69, C70: 0.1uF, SparkFun-Capacitors:0603
- removed D61, D62, D63, D64, D65, D66, D67, D68, D69, D70: 24V, SparkFun-DiscreteSemi:0603
- removed H61, H62, H63, H64, H65, H66, H67, H68, H69, H70: STAND-OFF, SparkFun-Hardware:STAND-OFF
- removed J61, J62, J63, J64, J65, J66, J67, J68, J69, J70: (no value), SparkFun-Connectors:1X03_NO_SILK
- removed JP241, JP242, JP243, JP244, JP245, JP246, JP247, JP248, JP249, JP250, JP251, JP252, JP253, JP254, JP255, JP256, JP257, JP258, JP259, JP260, JP261, JP262, JP263, JP264, JP265, JP266, JP267, JP268, JP269, JP270, JP271, JP272, JP273, JP274, JP275, JP276, JP277, JP278, JP279, JP280: FIDUCIALUFIDUCIAL, SparkFun:MICRO-FIDUCIAL
- removed LOGO181, LOGO184, LOGO187, LOGO190, LOGO193, LOGO196, LOGO199, LOGO202, LOGO205, LOGO208: OSHW-LOGOMINI, SparkFun-Aesthetics:OSHW-LOGO-MINI
- removed LOGO182, LOGO185, LOGO188, LOGO191, LOGO194, LOGO197, LOGO200, LOGO203, LOGO206, LOGO209: SFE_LOGO_NAME_FLAME.1_INCH, SparkFun-Aesthetics:SFE_LOGO_NAME_FLAME_.1
- removed LOGO183, LOGO186, LOGO189, LOGO192, LOGO195, LOGO198, LOGO201, LOGO204, LOGO207, LOGO210: SFE_LOGO_FLAME.1_INCH, SparkFun-Aesthetics:SFE_LOGO_FLAME_.1
- removed R61, R62, R63, R64, R65, R66, R67, R68, R69, R70: 47k, SparkFun-Resistors:0603
- removed U$541, U$550, U$559, U$568, U$577, U$586, U$595, U$604, U$613, U$622: (no value), output:PIR0
- removed U$542, U$551, U$560, U$569, U$578, U$587, U$596, U$605, U$614, U$623: (no value), output:170UA0
- removed U$543, U$552, U$561, U$570, U$579, U$588, U$597, U$606, U$615, U$624: (no value), output:1UA0
- removed U$544, U$553, U$562, U$571, U$580, U$589, U$598, U$607, U$616, U$625: (no value), output:BREAKOUT0
- removed U$545, U$554, U$563, U$572, U$581, U$590, U$599, U$608, U$617, U$626: (no value), output:#OUT#0
- removed U$546, U$555, U$564, U$573, U$582, U$591, U$600, U$609, U$618, U$627: (no value), output:#3V3#0
- removed U$547, U$556, U$565, U$574, U$583, U$592, U$601, U$610, U$619, U$628: (no value), output:#GND#0
- removed U$548, U$557, U$566, U$575, U$584, U$593, U$602, U$611, U$620, U$629: (no value), output:X0
- removed U$549, U$558, U$567, U$576, U$585, U$594, U$603, U$612, U$621, U$630: (no value), output:Y0
- removed U61, U62, U63, U64, U65, U66, U67, U68, U69, U70: EKMC4607112k, SparkFun-Sensors:TO-3
- moved C13 160.0 mm to (6.35, 25.4)
- moved C14 160.0 mm to (19.6, 25.4)
- moved D13 160.0 mm to (10.2, 25.4)
- moved D14 160.0 mm to (23.4, 25.4)
- moved H13 160.0 mm to (6.35, 41.1)
- moved H14 160.0 mm to (19.6, 41.1)
- moved J13 160.0 mm to (3.81, 23.4)
- moved J14 160.0 mm to (17.0, 23.4)
- moved LOGO37 160.0 mm to (11.2, 27.2)
- moved LOGO38 160.0 mm to (6.35, 36.1)
- moved LOGO39 160.0 mm to (1.46, 27.3)
- moved LOGO40 160.0 mm to (24.4, 27.2)
- moved LOGO41 160.0 mm to (19.6, 36.1)
- moved LOGO42 160.0 mm to (14.7, 27.3)
- moved R13 160.0 mm to (2.54, 25.4)
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Connections:
- removed net 3.3V60: C61.1, D61.2, J61.3, U61.VDD
- removed net 3.3V61: C62.1, D62.2, J62.3, U62.VDD
- removed net 3.3V62: C63.1, D63.2, J63.3, U63.VDD
- removed net 3.3V63: C64.1, D64.2, J64.3, U64.VDD
- removed net 3.3V64: C65.1, D65.2, J65.3, U65.VDD
- removed net 3.3V65: C66.1, D66.2, J66.3, U66.VDD
- removed net 3.3V66: C67.1, D67.2, J67.3, U67.VDD
- removed net 3.3V67: C68.1, D68.2, J68.3, U68.VDD
- removed net 3.3V68: C69.1, D69.2, J69.3, U69.VDD
- removed net 3.3V69: C70.1, D70.2, J70.3, U70.VDD
- removed net GND60: C61.2, D61.1, J61.1, R61.1, U61.GND
- removed net GND61: C62.2, D62.1, J62.1, R62.1, U62.GND
- removed net GND62: C63.2, D63.1, J63.1, R63.1, U63.GND
- removed net GND63: C64.2, D64.1, J64.1, R64.1, U64.GND
- removed net GND64: C65.2, D65.1, J65.1, R65.1, U65.GND
- removed net GND65: C66.2, D66.1, J66.1, R66.1, U66.GND
- removed net GND66: C67.2, D67.1, J67.1, R67.1, U67.GND
- removed net GND67: C68.2, D68.1, J68.1, R68.1, U68.GND
- removed net GND68: C69.2, D69.1, J69.1, R69.1, U69.GND
- removed net GND69: C70.2, D70.1, J70.1, R70.1, U70.GND
- removed net PIR_OUT60: J61.2, R61.2, U61.OUT
- removed net PIR_OUT61: J62.2, R62.2, U62.OUT
- removed net PIR_OUT62: J63.2, R63.2, U63.OUT
- removed net PIR_OUT63: J64.2, R64.2, U64.OUT
- removed net PIR_OUT64: J65.2, R65.2, U65.OUT
- removed net PIR_OUT65: J66.2, R66.2, U66.OUT
- removed net PIR_OUT66: J67.2, R67.2, U67.OUT
- removed net PIR_OUT67: J68.2, R68.2, U68.OUT
- removed net PIR_OUT68: J69.2, R69.2, U69.OUT
- removed net PIR_OUT69: J70.2, R70.2, U70.OUT
Routing:
- net PIR_OUT66: track 17.1 -> 0.00 mm, vias 1 -> 0
- net PIR_OUT61: track 17.1 -> 0.00 mm, vias 1 -> 0
- net PIR_OUT60: track 17.1 -> 0.00 mm, vias 1 -> 0
- net PIR_OUT65: track 17.1 -> 0.00 mm, vias 1 -> 0
- net PIR_OUT64: track 17.1 -> 0.00 mm, vias 1 -> 0
- net PIR_OUT63: track 17.1 -> 0.00 mm, vias 1 -> 0
- net PIR_OUT69: track 17.1 -> 0.00 mm, vias 1 -> 0
- net PIR_OUT68: track 17.1 -> 0.00 mm, vias 1 -> 0
- net PIR_OUT67: track 17.1 -> 0.00 mm, vias 1 -> 0
- net PIR_OUT62: track 17.1 -> 0.00 mm, vias 1 -> 0
- net 3.3V69: track 10.0 -> 0.00 mm
- net 3.3V68: track 10.0 -> 0.00 mm
- net 3.3V67: track 10.0 -> 0.00 mm
- net 3.3V62: track 10.0 -> 0.00 mm
- net 3.3V60: track 10.0 -> 0.00 mm
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- removed copper zone on layer 1, net GND60
- removed copper zone on layer 16, net GND60
- removed copper zone on layer 1, net GND61
- removed copper zone on layer 16, net GND61
- removed copper zone on layer 1, net GND62
- removed copper zone on layer 16, net GND62
- removed copper zone on layer 1, net GND63
- removed copper zone on layer 16, net GND63
- removed copper zone on layer 1, net GND64
- removed copper zone on layer 16, net GND64
- removed copper zone on layer 1, net GND65
- removed copper zone on layer 16, net GND65
- removed copper zone on layer 1, net GND66
- removed copper zone on layer 16, net GND66
- removed copper zone on layer 1, net GND67
- removed copper zone on layer 16, net GND67
- removed copper zone on layer 1, net GND68
- removed copper zone on layer 16, net GND68
- removed copper zone on layer 1, net GND69
- removed copper zone on layer 16, net GND69
Other:
- board size 204.5 x 124.2 mm -> 178.1 x 124.2 mm
